File: hardware/schematics/power_supply.kicad_sch (KiCad schematic)
At the start: 2 parts, among them U2 R-78E3.3-1.0

Commit message: Modified schematics to reflect design choices. Not finished
Parts:
- removed BT1: 12V_Battery, symbol Device:Battery_Cell
- removed U2: R-78E3.3-1.0, Converter_DCDC:Converter_DCDC_RECOM_R-78E-0.5_THT, symbol Converter_DCDC:R-78E3.3-1.0
Other:
- note removed: "12 V power for lock mechanism"
- note removed: "3.3V power for uC and NFC scanner"
